Commit message: update al5d model to modern configs

File: urdf/lynxmotion_al5d.xacro (robot description, xacro)
@@ -3,6 +3,4 @@
     <xacro:include filename="$(find lynxmotion_al5d_description)/urdf/lynxmotion_al5d_properties.urdf.xacro" />
     <!-- Base link comprising the board behind the robot and the cylinder at its bottom -->
-    <link name="world" />
-    <gazebo reference="world" />
     <link name="robot_support">
         <visual>
@@ -184,15 +182,4 @@
     </link>
     <!-- Adding joints -->
-    <joint name="world_to_robot" type="fixed">
-        <parent link="world" />
-        <child link="robot_support" />
-        <origin rpy="0 0 ${PI}" />
-        <dynamics damping="1.0" friction="0.8" />
-    </joint>
-    <joint name="camera_joint" type="fixed">
-        <parent link="world" />
-        <child link="camera_link" />
-        <origin xyz="0 0.17 ${camera_support_depth}" />
-    </joint>
    <joint name="Joint1" type="revolute">
         <parent link="robot_support" />

File: urdf/lynxmotion_al5d_properties.urdf.xacro (robot description, xacro)
@@ -15,5 +15,5 @@
     </material>
     <material name="BlueGrey">
-        <color rgba="1 87 155 1" />
+        <color rgba="0.004 0.34 0.61 1.0" />
     </material>
     <material name="Transparent">
@@ -59,9 +59,4 @@
     <xacro:property name="wrist_cylinder_length" value="0.005" />
     <xacro:property name="wrist_cylinder_radius" value="0.01" />
-    <xacro:property name="camera_support_depth" value="0.25" />
-    <xacro:property name="camera_support_size" value="0.01" />
-    <xacro:property name="camera_support_big_size" value="0.5" />
-    <xacro:property name="camera_support_to_base" value="0.1" />
-    <xacro:property name="camera_support_mass" value="0.2" />
     <!-- Adding macros for the inertial matrixes -->
     <xacro:macro name="inertial_matrix_cylinder" params="mass height radius">

Commit message: reorganized file with MoveIt Setup Assistant

File: urdf/lynxmotion_al5d.xacro (robot description, xacro)
@@ -1,4 +1,4 @@
 <?xml version="1.0" ?>
-<robot name="lynxmotion_al5d" xmlns:xacro="http://www.ros.org/wiki/xacro">
+<robot name="lynxmotion_al5d">
     <xacro:include filename="$(find lynxmotion_al5d_description)/urdf/lynxmotion_al5d_properties.urdf.xacro" />
     <!-- Base link comprising the board behind the robot and the cylinder at its bottom -->
@@ -18,5 +18,11 @@
         <xacro:inertial_matrix mass="${base_mass + board_mass}" ixx="3.6565e-7" ixy="-3.72e-9" ixz="1e-6" iyy="9.404e-8" iyz="4.375e-8" izz="4.1776e-7" xyz="0.000585 0.0602746 0.0170628" />
     </link>
-    <gazebo reference="robot_support" />
+    <gazebo reference="robot_support">
+        <plugin name="gazebo_ros_control" filename="libgazebo_ros_control.so">
+            <xacro:unless value="${robot_namespace == ''}">
+                <robotNamespace>($robot_namespace)</robotNamespace>
+            </xacro:unless>
+        </plugin>
+    </gazebo>
     <link name="robot_base_cylinder">
         <visual>
@@ -165,22 +171,6 @@
     </link>
     <gazebo reference="gripper_mov" />
-    <link name="camera_link">
-        <visual>
-            <geometry>
-                <box size="0.0001 0.0001 0.0001" />
-            </geometry>
-            <origin rpy="0 0 0" xyz="0 0 0" />
-            <material name="transparent">Gazebo/GreyTransparent</material>
-        </visual>
-        <collision>
-            <geometry>
-                <box size="0.0001 0.0001 0.0001" />
-            </geometry>
-            <origin rpy="0 0 0" xyz="0 0 0" />
-        </collision>
-        <xacro:inertial_matrix_bis mass="0.0005" />
-    </link>
     <!-- Adding joints -->
-   <joint name="Joint1" type="revolute">
+    <joint name="Joint1" type="revolute">
         <parent link="robot_support" />
         <child link="robot_base_cylinder" />
@@ -198,7 +188,7 @@
         <parent link="robot_base_top_box" />
         <child link="shoulder" />
-        <axis xyz="1 0 0"/>
+        <axis xyz="1 0 0" />
         <origin xyz="0 0.02 0.07" />
-        <limit effort="100" velocity="3" lower="0" upper="${PI}" />
+        <limit effort="100" lower="0" upper="${PI}" velocity="3" />
         <dynamics damping="1.0" friction="0.8" />
     </joint>
@@ -208,5 +198,5 @@
         <axis xyz="1 0 0" />
         <origin xyz="0 ${shoulder_to_elbow} 0" />
-        <limit effort="100" velocity="3" lower="${-PI}" upper="0" />
+        <limit effort="100" lower="${-PI}" upper="0" velocity="3" />
         <dynamics damping="1.0" friction="0.8" />
     </joint>
@@ -215,14 +205,14 @@
         <child link="wrist" />
         <axis xyz="1 0 0" />
-        <origin xyz="0 0.181 0.005" rpy="0 0 0"/>
-        <limit effort="40" velocity="3" lower="${-PI/2}" upper="${PI/2}" />
+        <origin rpy="0 0 0" xyz="0 0.181 0.005" />
+        <limit effort="40" lower="${-PI/2}" upper="${PI/2}" velocity="3" />
         <dynamics damping="5.0" friction="0.08" />
     </joint>
-   <joint name="Joint5" type="revolute">
+    <joint name="Joint5" type="revolute">
         <parent link="wrist" />
         <child link="gripper" />
         <axis xyz="0 -1 0" />
-        <origin xyz="0 0.04 0" rpy="0 0 ${PI}" />
-        <limit effort="100" velocity="3" lower="${-PI}" upper="${PI}" />
+        <origin rpy="0 0 ${PI}" xyz="0 0.04 0" />
+        <limit effort="100" lower="${-PI}" upper="${PI}" velocity="3" />
         <dynamics damping="1.0" friction="0.8" />
     </joint>
@@ -231,14 +221,14 @@
         <child link="right_finger" />
         <origin xyz="-0.005 -0.015 0" />
-        <limit effort="100" velocity="0.1" lower="0" upper="${gripper_base_width/2}" />
+        <limit effort="100" lower="0" upper="${gripper_base_width/2}" velocity="0.1" />
         <mimic joint="Gripper" multiplier="-0.5" offset="${gripper_base_width/2}" />
         <dynamics damping="1.0" friction="0.16" />
     </joint>
-   <joint name="left_finger_joint" type="prismatic">
+    <joint name="left_finger_joint" type="prismatic">
         <parent link="gripper" />
         <child link="left_finger" />
         <origin xyz="0.005 -0.015 0" />
         <axis xyz="-1 0 0" />
-        <limit effort="100" velocity="0.1" lower="0" upper="${gripper_base_width/2}" />
+        <limit effort="100" lower="0" upper="${gripper_base_width/2}" velocity="0.1" />
         <!-- Added an offset to fix issues in Rviz -->
         <mimic joint="right_finger_joint" offset="-0.0025" />
@@ -250,5 +240,5 @@
         <child link="gripper_mov" />
         <origin xyz="0.01 0  0" />
-        <limit lower="0" upper="${gripper_base_width}" effort="10" velocity="0.1" />
+        <limit effort="10" lower="0" upper="${gripper_base_width}" velocity="0.1" />
         <axis xyz="-1 0 0" />
         <dynamics damping="5.0" />
@@ -264,5 +254,5 @@
     <!-- ros_control plugin -->
     <gazebo>
-        <plugin name="gazebo_ros_control" filename="libgazebo_ros_control.so">
+        <plugin filename="libgazebo_ros_control.so" name="gazebo_ros_control">
             <robotNamespace>/lynxmotion_al5d</robotNamespace>
             <legacyModeNS>true</legacyModeNS>
@@ -271,34 +261,18 @@
     <!-- Setting the mimic joints plugin -->
     <xacro:mimic_joint_plugin_gazebo name_prefix="finger_right"
-    parent_joint="Gripper" mimic_joint="right_finger_joint" multiplier="-0.5"
-        has_pid="true" max_effort="10.0" offset="${gripper_base_width/2}" />
+        parent_joint="Gripper"
+        mimic_joint="right_finger_joint"
+        multiplier="-0.5"
+        has_pid="true"
+        max_effort="10.0"
+        offset="${gripper_base_width/2}"
+    />
     <xacro:mimic_joint_plugin_gazebo name_prefix="finger_left"
-    parent_joint="Gripper" has_pid="true"  mimic_joint="left_finger_joint" multiplier="-0.5" max_effort="10.0" offset="${gripper_base_width/2}" />
-    <gazebo reference="camera_link">
-        <sensor name="external_camera" type="camera">
-            <update_rate>1.0</update_rate>
-            <camera name="camera_top">
-                <horizontal_fov>1.2</horizontal_fov>
-                <pose>0 0 0 3.1415 1.5708 -1.5708</pose>
-                <image>
-                    <width>640</width>
-                    <height>480</height>
-                    <format>R8G8B8</format>
-                </image>
-                <clip>
-                    <near>0.01</near>
-                    <far>0.3</far>
-                </clip>
-            </camera>
-            <plugin filename="libgazebo_ros_camera.so" name="camera_controller">
-                <robotNamespace>/lynxmotion_al5d</robotNamespace>
-                <alwaysOn>true</alwaysOn>
-                <updateRate>1.0</updateRate>
-                <cameraName>external_vision</cameraName>
-                <imageToPIcName>image_raw</imageToPIcName>
-                <cameraInfoToPIcName>camera_info</cameraInfoToPIcName>
-                <frameName>camera_link</frameName>
-            </plugin>
-        </sensor>
-    </gazebo>
+        parent_joint="Gripper"
+        has_pid="true"
+        mimic_joint="left_finger_joint"
+        multiplier="-0.5"
+        max_effort="10.0"
+        offset="${gripper_base_width/2}"
+    />
 </robot>

Commit message: clean up

File: urdf/lynxmotion_al5d.xacro (robot description, xacro)
@@ -18,11 +18,5 @@
         <xacro:inertial_matrix mass="${base_mass + board_mass}" ixx="3.6565e-7" ixy="-3.72e-9" ixz="1e-6" iyy="9.404e-8" iyz="4.375e-8" izz="4.1776e-7" xyz="0.000585 0.0602746 0.0170628" />
     </link>
-    <gazebo reference="robot_support">
-        <plugin name="gazebo_ros_control" filename="libgazebo_ros_control.so">
-            <xacro:unless value="${robot_namespace == ''}">
-                <robotNamespace>($robot_namespace)</robotNamespace>
-            </xacro:unless>
-        </plugin>
-    </gazebo>
+    <gazebo reference="robot_support" />
     <link name="robot_base_cylinder">
         <visual>
@@ -246,10 +240,10 @@
     </joint>
     <!-- Setting transmissions -->
-    <xacro:transmission_block joint_name="Joint1"/>
-    <xacro:transmission_block joint_name="Joint2"/>
-    <xacro:transmission_block joint_name="Joint3"/>
-    <xacro:transmission_block joint_name="Joint4"/>
-    <xacro:transmission_block joint_name="Joint5"/>
-    <xacro:transmission_block joint_name="Gripper"/>
+    <xacro:transmission_block joint_name="Joint1" idx="1" />
+    <xacro:transmission_block joint_name="Joint2" idx="2" />
+    <xacro:transmission_block joint_name="Joint3" idx="3" />
+    <xacro:transmission_block joint_name="Joint4" idx="4" />
+    <xacro:transmission_block joint_name="Joint5" idx="5" />
+    <xacro:transmission_block joint_name="Gripper" idx="6" />
     <!-- ros_control plugin -->
     <gazebo>

File: urdf/lynxmotion_al5d_properties.urdf.xacro (robot description, xacro)
@@ -88,7 +88,10 @@
    <xacro:macro name="mimic_joint_plugin_gazebo" params="name_prefix parent_joint mimic_joint has_pid:=false multiplier:=1.0 offset:=0 sensitiveness:=0.0 max_effort:=1.0 robot_namespace:=''">
     <gazebo>
-      <plugin name="${name_prefix}mimic_joint_plugin" filename="libroboticsgroup_gazebo_mimic_joint_plugin.so">
+      <plugin name="${name_prefix}_mimic_joint_plugin" filename="libroboticsgroup_gazebo_mimic_joint_plugin.so">
         <joint>${parent_joint}</joint>
         <mimicJoint>${mimic_joint}</mimicJoint>
+        <xacro:unless value="${robot_namespace == ''}">
+          <robotNamespace>($robot_namespace)</robotNamespace>
+        </xacro:unless>
         <xacro:if value="${has_pid}">
           <hasPID />
@@ -98,18 +101,16 @@
         <sensitiveness>${sensitiveness}</sensitiveness>
         <maxEffort>${max_effort}</maxEffort>
-        <xacro:unless value="${robot_namespace == ''}">
-          <robotNamespace>($robot_namespace)</robotNamespace>
-        </xacro:unless>
       </plugin>
     </gazebo>
   </xacro:macro>
-    <xacro:macro name="transmission_block" params="joint_name">
-        <transmission name="tran1">
+    <xacro:macro name="transmission_block" params="joint_name idx">
+        <transmission name="tran${idx}">
             <type>transmission_interface/SimpleTransmission</type>
             <joint name="${joint_name}">
                 <hardwareInterface>hardware_interface/PositionJointInterface</hardwareInterface>
             </joint>
-            <actuator name="motor1">
+            <actuator name="motor${idx}">
                 <mechanicalReduction>1</mechanicalReduction>
+                <hardwareInterface>hardware_interface/EffortJointInterface</hardwareInterface>
             </actuator>
         </transmission>
