Commit message: reorganized compilation to put all packages into 1 directory. introduced linker issue in pick_place package (tmrw problem).

File: lynxmotion_al5d_description/urdf/lynxmotion_al5d_properties.urdf.xacro (robot description, xacro)
@@ -24,8 +24,8 @@
     <xacro:property name="board_size" value="0.03" />
     <xacro:property name="board_height" value="0.005" />
-    <xacro:property name="board_mass" value="0.3" />
+    <xacro:property name="board_mass" value="0.5" />
     <xacro:property name="base_radius" value="0.025" />
     <xacro:property name="base_height" value="0.04" />
-    <xacro:property name="base_mass" value="2" />
+    <xacro:property name="base_mass" value="4" />
     <xacro:property name="top_box_width" value="0.03" />
     <xacro:property name="top_box_height" value="0.025" />

File: lynxmotion_al5d_moveit/config/gazebo_lynxmotion_al5d.urdf (robot description, URDF)
Before this commit: robot lynxmotion_al5d, 10 links, 9 joints
Links:
- link robot_support: mass 2.3 -> 23
